File: HX711.sch (KiCad schematic (older format))
At the start: 8 parts, among them Q1 Q_PNP_BEC, U3 HX711

Commit message: update files
Parts:
- C3: value 0.1uF -> 100nF
Changed lines of the file:
@@
 P 3650 3850
 F 0 "C3" H 3535 3804 50  0000 R CNN
-F 1 "0.1uF" H 3535 3895 50  0000 R CNN
+F 1 "100nF" H 3535 3895 50  0000 R CNN
 F 2 "Capacitor_THT:CP_Radial_D4.0mm_P1.50mm" H 3688 3700 50  0001 C CNN
 F 3 "~" H 3650 3850 50  0001 C CNN

Commit message: update files
Parts:
- C1, C2, C3: footprint Capacitor_THT:CP_Radial_D4.0mm_P1.50mm -> Capacitor_SMD:C_1206_3216Metric_Pad1.33x1.80mm_HandSolder
- Q1: footprint Package_TO_SOT_SMD:SOT-23 -> Connector_PinHeader_2.54mm:PinHeader_1x02_P2.54mm_Vertical
Changed lines of the file:
@@
 F 0 "C1" H 2935 1704 50  0000 R CNN
 F 1 "10uF" H 2935 1795 50  0000 R CNN
-F 2 "Capacitor_THT:CP_Radial_D4.0mm_P1.50mm" H 3088 1600 50  0001 C CNN
+F 2 "Capacitor_SMD:C_1206_3216Metric_Pad1.33x1.80mm_HandSolder" H 3088 1600 50  0001 C CNN
 F 3 "~" H 3050 1750 50  0001 C CNN
 	1    3050 1750
@@
 Wire Wire Line
 	5300 2700 5400 2700
-Wire Wire Line
-	5400 2700 5400 2750
 Text HLabel 6550 3250 2    50   Input ~ 0
 VCC
@@
 F 0 "C2" H 3565 4646 50  0000 L CNN
 F 1 "100nF" H 3565 4555 50  0000 L CNN
-F 2 "Capacitor_THT:CP_Radial_D4.0mm_P1.50mm" H 3488 4450 50  0001 C CNN
+F 2 "Capacitor_SMD:C_1206_3216Metric_Pad1.33x1.80mm_HandSolder" H 3488 4450 50  0001 C CNN
 F 3 "~" H 3450 4600 50  0001 C CNN
 	1    3450 4600
@@
 F 0 "C3" H 3535 3804 50  0000 R CNN
 F 1 "100nF" H 3535 3895 50  0000 R CNN
-F 2 "Capacitor_THT:CP_Radial_D4.0mm_P1.50mm" H 3688 3700 50  0001 C CNN
+F 2 "Capacitor_SMD:C_1206_3216Metric_Pad1.33x1.80mm_HandSolder" H 3688 3700 50  0001 C CNN
 F 3 "~" H 3650 3850 50  0001 C CNN
 	1    3650 3850
@@
 F 0 "Q1" H 3941 1954 50  0000 L CNN
 F 1 "Q_PNP_BEC" H 3941 2045 50  0000 L CNN
-F 2 "Package_TO_SOT_SMD:SOT-23" H 3950 2100 50  0001 C CNN
+F 2 "Connector_PinHeader_2.54mm:PinHeader_1x02_P2.54mm_Vertical" H 3950 2100 50  0001 C CNN
 F 3 "~" H 3750 2000 50  0001 C CNN
 	1    3750 2000
@@
 	5550 2800 5550 2750
 Wire Wire Line
+	6550 2800 6150 2800
+Wire Wire Line
+	6150 2800 6150 2750
+Wire Notes Line
+	1950 2750 2250 2750
+Wire Notes Line
+	2250 2750 2250 3400
+Wire Notes Line
+	2250 3400 1950 3400
+Wire Notes Line
+	1950 3400 1950 2750
+Wire Wire Line
+	5400 2700 5400 2750
+Wire Wire Line
+	6150 2750 5550 2750
+Wire Wire Line
 	5550 2750 5400 2750
+Connection ~ 5550 2750
 Connection ~ 5400 2750
 Wire Wire Line
 	5400 2750 5400 2800
-Wire Wire Line
-	6550 2800 6150 2800
-Wire Wire Line
-	6150 2800 6150 2750
-Wire Wire Line
-	6150 2750 5550 2750
-Connection ~ 5550 2750
-Wire Notes Line
-	1950 2750 2250 2750
-Wire Notes Line
-	2250 2750 2250 3400
-Wire Notes Line
-	2250 3400 1950 3400
-Wire Notes Line
-	1950 3400 1950 2750
 $EndSCHEMATC

Commit message: Update files
Parts:
- added C5: 10uF, Capacitor_SMD:C_1206_3216Metric_Pad1.33x1.80mm_HandSolder, symbol Device:C
- added C6: 100nF, Capacitor_SMD:C_1206_3216Metric_Pad1.33x1.80mm_HandSolder, symbol Device:C
- added R11: 1.2k, Resistor_SMD:R_1206_3216Metric, symbol Device:R
- Q1: footprint Connector_PinHeader_2.54mm:PinHeader_1x02_P2.54mm_Vertical -> Package_TO_SOT_SMD:SOT-23
Connections:
- net E+: now also C5.2
- net E-: now also C5.1
- net GND: no longer U3.10 (INB+), U3.9 (INB-)
- new net: C6.1, R11.2, U3.10 (INB+)
- new net B+: R11.1
- new net B-: C6.2, U3.9 (INB-)
Changed lines of the file:
@@
 	-1   0    0    1
 $EndComp
-$Comp
-L PCB_TP_Prof-rescue:GND #PWR02
-U 1 1 602086B3
-P 5450 3450
-F 0 "#PWR02" H 5450 3450 30  0001 C CNN
-F 1 "GND" H 5450 3380 30  0001 C CNN
-F 2 "" H 5450 3450 60  0000 C CNN
-F 3 "" H 5450 3450 60  0000 C CNN
-	1    5450 3450
-	1    0    0    -1
-$EndComp
-Wire Wire Line
-	5450 3450 5450 3300
-Wire Wire Line
-	5450 3300 5300 3300
-Wire Wire Line
-	5450 3300 5450 3200
-Wire Wire Line
-	5450 3200 5300 3200
-Connection ~ 5450 3300
 Connection ~ 5600 1550
 $Comp
@@
 F 0 "Q1" H 3941 1954 50  0000 L CNN
 F 1 "Q_PNP_BEC" H 3941 2045 50  0000 L CNN
-F 2 "Connector_PinHeader_2.54mm:PinHeader_1x02_P2.54mm_Vertical" H 3950 2100 50  0001 C CNN
+F 2 "Package_TO_SOT_SMD:SOT-23" H 3950 2100 50  0001 C CNN
 F 3 "~" H 3750 2000 50  0001 C CNN
 	1    3750 2000
@@
 	2450 2850 2200 2850
 Connection ~ 3650 2800
-Wire Wire Line
-	3650 2800 2450 2800
 Wire Wire Line
 	3050 1900 3050 2150
@@
 Wire Wire Line
 	3000 3150 3000 4250
-Wire Wire Line
-	3650 3600 3200 3600
-Wire Wire Line
-	3200 3600 3200 3000
-Wire Wire Line
-	3200 3000 2200 3000
 $Comp
 L PCB_TP_Prof-rescue:GND #PWR0101
@@
 Wire Wire Line
 	5400 2750 5400 2800
+$Comp
+L Device:C C5
+U 1 1 606316D8
+P 3300 3150
+F 0 "C5" H 3185 3104 50  0000 R CNN
+F 1 "10uF" H 3185 3195 50  0000 R CNN
+F 2 "Capacitor_SMD:C_1206_3216Metric_Pad1.33x1.80mm_HandSolder" H 3338 3000 50  0001 C CNN
+F 3 "~" H 3300 3150 50  0001 C CNN
+	1    3300 3150
+	-1   0    0    1
+$EndComp
+Wire Wire Line
+	3100 3600 3100 3000
+Wire Wire Line
+	3100 3000 2200 3000
+Wire Wire Line
+	2450 2800 3300 2800
+Wire Wire Line
+	3100 3600 3300 3600
+Wire Wire Line
+	3300 3300 3300 3600
+Connection ~ 3300 3600
+Wire Wire Line
+	3300 3600 3650 3600
+Wire Wire Line
+	3300 3000 3300 2800
+Connection ~ 3300 2800
+Wire Wire Line
+	3300 2800 3650 2800
+$Comp
+L Device:R R11
+U 1 1 60639E3C
+P 6050 3850
+F 0 "R11" V 5843 3850 50  0000 C CNN
+F 1 "1.2k" V 5934 3850 50  0000 C CNN
+F 2 "Resistor_SMD:R_1206_3216Metric" V 5980 3850 50  0001 C CNN
+F 3 "~" H 6050 3850 50  0001 C CNN
+	1    6050 3850
+	-1   0    0    1
+$EndComp
+Wire Wire Line
+	5850 3200 5850 3550
+Wire Wire Line
+	5300 3200 5850 3200
+$Comp
+L Device:C C6
+U 1 1 6063C369
+P 5550 3850
+F 0 "C6" H 5665 3896 50  0000 L CNN
+F 1 "100nF" H 5665 3805 50  0000 L CNN
+F 2 "Capacitor_SMD:C_1206_3216Metric_Pad1.33x1.80mm_HandSolder" H 5588 3700 50  0001 C CNN
+F 3 "~" H 5550 3850 50  0001 C CNN
+	1    5550 3850
+	1    0    0    -1
+$EndComp
+Wire Wire Line
+	5550 3700 5550 3550
+Wire Wire Line
+	5550 3550 5850 3550
+Wire Wire Line
+	6050 3550 6050 3700
+Wire Wire Line
+	5300 3300 5350 3300
+Wire Wire Line
+	5350 3300 5350 4100
+Wire Wire Line
+	5350 4100 5550 4100
+Wire Wire Line
+	5550 4100 5550 4000
+Wire Wire Line
+	6050 4000 6050 4400
+Wire Wire Line
+	5550 4100 5550 4400
+Connection ~ 5550 4100
+Text HLabel 6050 4400 3    50   Input ~ 0
+B+
+Text HLabel 5550 4400 3    50   Input ~ 0
+B-
+Wire Wire Line
+	6050 3550 5850 3550
+Connection ~ 5850 3550
 $EndSCHEMATC
