File: Conector.sch (KiCad schematic (older format))
At the start: 1 part

Commit message: update files
Connections:
- net +3.3V renamed +3.3V_P1
- net +3.3V_P1: no longer XA1.41 (+3.3V)
- net +5V renamed +5V_P1
- net +5V_P1: no longer XA1.42 (+5V)
- new net +3.3V_P2: XA1.41 (+3.3V)
- new net +5V_P2: XA1.42 (+5V)
Changed lines of the file:
@@
 NoConn ~ 7600 3600
 Text HLabel 3200 2300 0    50   UnSpc ~ 0
-+3.3V
++3.3V_P2
 Text HLabel 4900 2300 2    50   UnSpc ~ 0
-+5V
++5V_P2
 Text HLabel 9050 2300 2    50   UnSpc ~ 0
-+5V
++5V_P1
 Text HLabel 7350 2300 0    50   UnSpc ~ 0
-+3.3V
++3.3V_P1
 Wire Wire Line
 	7600 2300 7350 2300
@@
 Wire Wire Line
 	3200 2300 3450 2300
+Text HLabel 9450 4200 2    50   UnSpc ~ 0
+GND
+Wire Wire Line
+	9450 4200 9200 4200
 $EndSCHEMATC

Commit message: update files
Connections:
- net CAN_RD-GPIO33: now reaches XA1.27 (canRD)
- net CAN_TD-GPIO32: now reaches XA1.29 (canTD)
- net T_COL1-GPIO30: now reaches XA1.31 (tecCOL1)
- net T_FIL0-GPIO25: now reaches XA1.33 (tecF0)
- net T_FIL3-GPIO28: now reaches XA1.35 (tecF3)
- net T_FIL2-GPIO27: now reaches XA1.37 (tecF2)
- net T_COL0-GPIO29: now reaches XA1.39 (tecCOL0)
- net RXD1-GPIO21: now reaches XA1.44 (ethRXD1)
- net TX_EN-GPIO19: now reaches XA1.46 (ethTXEN)
- no-connect marks 35 -> 26
Changed lines of the file:
@@
 NoConn ~ 4650 2700
 NoConn ~ 4650 2600
-NoConn ~ 4650 2500
-NoConn ~ 4650 2400
 NoConn ~ 3450 3300
 $Comp
@@
 NoConn ~ 7600 2500
 NoConn ~ 7600 2600
-NoConn ~ 7600 4200
-NoConn ~ 7600 4100
-NoConn ~ 7600 4000
-NoConn ~ 7600 3900
-NoConn ~ 7600 3800
 NoConn ~ 8800 4000
 NoConn ~ 8800 3900
@@
 Wire Wire Line
 	7350 3500 7600 3500
-NoConn ~ 7600 3700
-NoConn ~ 7600 3600
 Text HLabel 3200 2300 0    50   UnSpc ~ 0
 +3.3V_P2
@@
 Wire Wire Line
 	9450 4200 9200 4200
+Text HLabel 7350 3800 0    50   BiDi ~ 0
+T_COL1-GPIO30
+Wire Wire Line
+	7350 3800 7600 3800
+Text HLabel 7350 3900 0    50   BiDi ~ 0
+T_FIL0-GPIO25
+Wire Wire Line
+	7350 3900 7600 3900
+Text HLabel 7350 4200 0    50   BiDi ~ 0
+T_COL0-GPIO29
+Wire Wire Line
+	7350 4200 7600 4200
+Text HLabel 7350 4100 0    50   BiDi ~ 0
+T_FIL2-GPIO27
+Wire Wire Line
+	7350 4100 7600 4100
+Text HLabel 7350 4000 0    50   BiDi ~ 0
+T_FIL3-GPIO28
+Wire Wire Line
+	7350 4000 7600 4000
+Text HLabel 7350 3600 0    50   BiDi ~ 0
+CAN_RD-GPIO33
+Wire Wire Line
+	7350 3600 7600 3600
+Text HLabel 7350 3700 0    50   BiDi ~ 0
+CAN_TD-GPIO32
+Wire Wire Line
+	7350 3700 7600 3700
+Text HLabel 4900 2400 2    50   BiDi ~ 0
+RXD1-GPIO21
+Wire Wire Line
+	4900 2400 4650 2400
+Text HLabel 4900 2500 2    50   BiDi ~ 0
+TX_EN-GPIO19
+Wire Wire Line
+	4900 2500 4650 2500
 $EndSCHEMATC

Commit message: Update files + gerbers
Connections:
- net GNDA: now reaches XA1.18 (GNDA)
- no-connect marks 26 -> 25
Changed lines of the file:
@@
 NoConn ~ 8800 4000
 NoConn ~ 8800 3900
-NoConn ~ 8800 3100
 NoConn ~ 8800 3000
 NoConn ~ 8800 2900
@@
 Wire Wire Line
 	4900 2500 4650 2500
+Text HLabel 8900 3100 2    50   UnSpc ~ 0
+GNDA
+Wire Wire Line
+	8900 3100 8800 3100
 $EndSCHEMATC
