File: PCB_TP_Prof.sch (KiCad schematic (older format))
At the start: 8 parts, among them J1 Conn_01x04_Female, J2 Conn_01x01_Male

Commit message: update files
Parts:
- removed J1: Conn_01x04_Female, Connector_PinHeader_2.54mm:PinHeader_1x04_P2.54mm_Vertical, symbol Connector:Conn_01x04_Female
- removed J2: Conn_01x01_Male, Connector_PinHeader_2.54mm:PinHeader_1x01_P2.54mm_Vertical, symbol Connector:Conn_01x01_Male
- added J2: Conn_01x12_Female, Connector_PinHeader_2.54mm:PinHeader_1x12_P2.54mm_Vertical, symbol Connector:Conn_01x12_Female
Connections:
- wire segments 34 -> 68
- no-connect marks 0 -> 1
Other:
- note added: "DT y SCK pueden ir a \ncualquier GPIO de la EDU-CIAA"
- note added: "LL\n"
- note added: "LR"
- note added: "UL\n"
- note added: "UR\n"
- moved on the sheet: JP1, R4, U_MUX1

Commit message: update files
Parts:
- removed U_DEMUX1, U_MUX1: CD74HC4067M, Package_SO:SOIC-24W_7.5x15.4mm_P1.27mm, symbol 74xx:CD74HC4067M
- added J1, J3: Conn_01x16_Female, Connector_PinHeader_2.54mm:PinHeader_1x16_P2.54mm_Vertical, symbol Connector:Conn_01x16_Female
- added J4, J5, J6: Conn_01x01_Male, Connector_PinHeader_2.54mm:PinHeader_1x01_P2.54mm_Vertical, symbol Connector:Conn_01x01_Male
- added JP3, JP4, JP5, JP6, JP7, JP8: Jumper, Connector_PinHeader_2.54mm:PinHeader_1x02_P2.54mm_Vertical, symbol Device:Jumper
- added U_DEMUX1, U_MUX1: CD74HC4067SM, Package_SO:SSOP-24_5.3x8.2mm_P0.65mm, symbol 74xx:CD74HC4067SM
Connections:
- net +3V3: now also JP4.1
- net +5V: now also JP1.2, JP2.2, JP3.2
- net Conector-EDU_CIAA/232_RX: now also JP6.1
- net Conector-EDU_CIAA/232_TX: now also JP7.1
- net Conector-EDU_CIAA/CH3: now also U_MUX1.1 (COM)
- net Conector-EDU_CIAA/GPIO1: now also U_DEMUX1.10 (S0)
- net Conector-EDU_CIAA/GPIO3: now also U_DEMUX1.11 (S1)
- net Conector-EDU_CIAA/GPIO5: now also U_DEMUX1.14 (S2)
- net Conector-EDU_CIAA/GPIO7: now also U_DEMUX1.13 (S3)
- net Conector-EDU_CIAA/GPIO8: now also U_DEMUX1.1 (COM)
- net GND: now also J1.15 (Pin_15), J1.16 (Pin_16), J3.13 (Pin_13), J3.14 (Pin_14), J3.15 (Pin_15), J3.16 (Pin_16), J6.1 (Pin_1), U_DEMUX1.12 (GND), U_DEMUX1.16 (I15), U_DEMUX1.17 (I14), U_MUX1.12 (GND), U_MUX1.16 (I15), U_MUX1.17 (I14), U_MUX1.18 (I13), U_MUX1.19 (I12)
- net HX711/DT: now also JP8.1
- net HX711/SCK: now also JP5.1
- net NodeMCU/RST: now also J4.1 (Pin_1)
- net at R4.1: now also U_DEMUX1.15 (~E)
- net at JP1.1: now also U_DEMUX1.24 (VCC)
- net at R5.1: now also U_MUX1.15 (~E)
- net at JP2.1: now also U_MUX1.24 (VCC)
- new net: J1.1 (Pin_1), U_DEMUX1.9 (I0)
- new net: J1.10 (Pin_10), U_DEMUX1.22 (I9)
- new net: J1.11 (Pin_11), U_DEMUX1.21 (I10)
- new net: J1.12 (Pin_12), U_DEMUX1.20 (I11)
- new net: J1.13 (Pin_13), U_DEMUX1.19 (I12)
- new net: J1.14 (Pin_14), U_DEMUX1.18 (I13)
- new net: J1.2 (Pin_2), U_DEMUX1.8 (I1)
- new net: J1.3 (Pin_3), U_DEMUX1.7 (I2)
- new net: J1.4 (Pin_4), U_DEMUX1.6 (I3)
- new net: J1.5 (Pin_5), U_DEMUX1.5 (I4)
- new net: J1.6 (Pin_6), U_DEMUX1.4 (I5)
- new net: J1.7 (Pin_7), U_DEMUX1.3 (I6)
- new net: J1.8 (Pin_8), U_DEMUX1.2 (I7)
- new net: J1.9 (Pin_9), U_DEMUX1.23 (I8)
- new net: J3.1 (Pin_1), U_MUX1.9 (I0)
- new net: J3.10 (Pin_10), U_MUX1.22 (I9)
- new net: J3.11 (Pin_11), U_MUX1.21 (I10)
- new net: J3.12 (Pin_12), U_MUX1.20 (I11)
- new net: J3.2 (Pin_2), U_MUX1.8 (I1)
- new net: J3.3 (Pin_3), U_MUX1.7 (I2)
- new net: J3.4 (Pin_4), U_MUX1.6 (I3)
- new net: J3.5 (Pin_5), U_MUX1.5 (I4)
- new net: J3.6 (Pin_6), U_MUX1.4 (I5)
- new net: J3.7 (Pin_7), U_MUX1.3 (I6)
- new net: J3.8 (Pin_8), U_MUX1.2 (I7)
- new net: J3.9 (Pin_9), U_MUX1.23 (I8)
- new net Conector-EDU_CIAA/RXD1-GPIO21: JP5.2
- new net Conector-EDU_CIAA/TX_EN-GPIO19: JP8.2
- new net Conector-EDU_CIAA/T_COL0-GPIO29: U_MUX1.13 (S3)
- new net Conector-EDU_CIAA/T_FIL0-GPIO25: U_MUX1.10 (S0)
- new net Conector-EDU_CIAA/T_FIL2-GPIO27: U_MUX1.14 (S2)
- new net Conector-EDU_CIAA/T_FIL3-GPIO28: U_MUX1.11 (S1)
- new net HX711/VCC: JP3.1
- new net NodeMCU/+3V3: JP4.2
- new net NodeMCU/GPIO0-D3: J5.1 (Pin_1)
- new net NodeMCU/RX: JP7.2
- new net NodeMCU/TX: JP6.2
- no-connect marks 1 -> 0
Other:
- note added: "Conectarlo a +3V3\ndel NodeMCU \npara programarlo"
- note added: "Para conectar al NodeMCU y asi \npoder programar el ESP12\n"
- note added: "Pines conectados \nal velostato (in)\n"
- note added: "Pines conectados \nal velostato (out)\n"
- note added: "Ponemos los 16 pines por las dudas\no ponemos los que sabemos que \nvamos a usar?\n"
- note added: "These devices have an enable \ncontrol which when high will \ndisable all switches to their \n“off” state."
- moved on the sheet: JP1, JP2, R4, R5

Commit message: Update files
Changed lines of the file:
@@
 	10000 5250 9700 5250
 Connection ~ 9900 5900
-Wire Wire Line
-	9900 5900 9850 5900
 $EndSCHEMATC

Commit message: Update files
Connections:
- no-connect marks 0 -> 2
Changed lines of the file:
@@
 F8 "VCC" I R 3650 2650 50
 F9 "GND" I R 3650 2100 50
+F10 "B+" I L 2450 2850 50
+F11 "B-" I L 2450 3000 50
 $EndSheet
 $Sheet
@@
 	10000 5250 9700 5250
 Connection ~ 9900 5900
+NoConn ~ 2300 2850
+Wire Wire Line
+	2300 2850 2450 2850
+NoConn ~ 2300 3000
+Wire Wire Line
+	2300 3000 2450 3000
 $EndSCHEMATC

Commit message: Update files + gerbers
Parts:
- added C7, C8: C, Capacitor_SMD:C_1206_3216Metric_Pad1.33x1.80mm_HandSolder, symbol Device:C
- added R12, R13, R14, R15, R16, R17, R18, R19, R20, R21, R22, R23, R24, R25, R26, R27: 1k, Resistor_SMD:R_1206_3216Metric, symbol Device:R
Connections:
- net GND: now also C7.2; no longer J3.13 (Pin_13), J3.14 (Pin_14), J3.15 (Pin_15), J3.16 (Pin_16), R5.2, U_MUX1.12 (GND), U_MUX1.16 (I15), U_MUX1.17 (I14), U_MUX1.18 (I13), U_MUX1.19 (I12)
- net at JP1.1, U_DEMUX1.24 (VCC): now also C7.1
- net at JP2.1, U_MUX1.24 (VCC): now also C8.2
- net at J3.1 (Pin_1), U_MUX1.9 (I0): now also R27.1
- net at J3.10 (Pin_10), U_MUX1.22 (I9): now also R18.1
- net at J3.11 (Pin_11), U_MUX1.21 (I10): now also R17.1
- net at J3.12 (Pin_12), U_MUX1.20 (I11): now also R16.1
- net at J3.2 (Pin_2), U_MUX1.8 (I1): now also R26.1
- net at J3.3 (Pin_3), U_MUX1.7 (I2): now also R25.1
- net at J3.4 (Pin_4), U_MUX1.6 (I3): now also R24.1
- net at J3.5 (Pin_5), U_MUX1.5 (I4): now also R23.1
- net at J3.6 (Pin_6), U_MUX1.4 (I5): now also R22.1
- net at J3.7 (Pin_7), U_MUX1.3 (I6): now also R21.1
- net at J3.8 (Pin_8), U_MUX1.2 (I7): now also R20.1
- net at J3.9 (Pin_9), U_MUX1.23 (I8): now also R19.1
- new net: J3.13 (Pin_13), R15.1, U_MUX1.19 (I12)
- new net: J3.14 (Pin_14), R14.1, U_MUX1.18 (I13)
- new net: J3.15 (Pin_15), R13.1, U_MUX1.17 (I14)
- new net: J3.16 (Pin_16), R12.1, U_MUX1.16 (I15)
- new net GNDA: C8.1, R12.2, R13.2, R14.2, R15.2, R16.2, R17.2, R18.2, R19.2, R20.2, R21.2, R22.2, R23.2, R24.2, R25.2, R26.2, R27.2, R5.2, U_MUX1.12 (GND)
Other:
- note added: "En caso de no usar los ultimos 4 pines, \nconectarlos directamente a GND\n"
- moved on the sheet: J3, JP1, JP2, R5, U_MUX1
