File: PCB_TP_Prof.kicad_pcb (KiCad board)
At the start: 2 copper layers, 85.9 x 91.7 mm, 19 parts, among them J1 Conn_01x04_Female, J2 Conn_01x01_Male, Q1 Q_PNP_BEC, U2 ESP-12E, U3 HX711

Commit message: update files
Parts:
- removed J1: Conn_01x04_Female, Connector_PinHeader_2.54mm:PinHeader_1x04_P2.54mm_Vertical
- added JP3: Jumper, Connector_PinHeader_2.54mm:PinHeader_1x02_P2.54mm_Vertical, F.Cu at (85.2, 64.8)
- added JP4: Jumper, Connector_PinHeader_2.54mm:PinHeader_1x02_P2.54mm_Vertical, F.Cu at (89.9, 64.8)
- added JP5: Jumper, Connector_PinHeader_2.54mm:PinHeader_1x02_P2.54mm_Vertical, F.Cu at (85.2, 72.0)
- added JP6: Jumper, Connector_PinHeader_2.54mm:PinHeader_1x02_P2.54mm_Vertical, F.Cu at (89.9, 72.0)
- added JP7: Jumper, Connector_PinHeader_2.54mm:PinHeader_1x02_P2.54mm_Vertical, F.Cu at (94.5, 64.8)
- added JP8: Jumper, Connector_PinHeader_2.54mm:PinHeader_1x02_P2.54mm_Vertical, F.Cu at (99.2, 64.8)
- added MP?: Plantilla_EDU-CIAA, Poncho_Esqueleto:Plantilla_EDU-CIAA, F.Cu at (133.9, 97.3)
- added R10: 10k, Resistor_SMD:R_1206_3216Metric, F.Cu at (100.6, 71.3)
- added R7: 10k, Resistor_SMD:R_1206_3216Metric, F.Cu at (95.0, 71.3)
- added R8: 10k, Resistor_SMD:R_1206_3216Metric, F.Cu at (95.0, 74.6)
- added R9: 10k, Resistor_SMD:R_1206_3216Metric, F.Cu at (91.3, 78.5)
- added SW1: SW_MEC_5G, Button_Switch_THT:SW_PUSH_6mm, F.Cu at (74.4, 64.5)
- added SW2: SW_MEC_5G, Button_Switch_THT:SW_PUSH_6mm, F.Cu at (74.4, 73.1)
- C3: value 0.1uF -> 100nF
- J2: value Conn_01x01_Male -> Conn_01x12_Female; footprint Connector_PinHeader_2.54mm:PinHeader_1x01_P2.54mm_Vertical -> Connector_PinHeader_2.54mm:PinHeader_1x12_P2.54mm_Vertical
- R6: value R -> 10k
- moved J2 179.2 mm to (77.5, 90.2)
- moved U3 156.6 mm to (89.6, 121.0)
- moved JP1 149.0 mm to (102.3, 143.8)
- moved JP2 149.0 mm to (107.0, 131.5)
- moved R5 149.0 mm to (77.0, 147.8)
- moved U_DEMUX1 149.0 mm to (93.5, 137.7)
- moved U_MUX1 149.0 mm to (80.6, 137.7)
- moved R4 149.0 mm to (82.6, 147.8)
- moved C1 146.2 mm to (89.1, 94.2)
- moved C2 146.2 mm to (89.1, 99.8)
- moved C3 146.2 mm to (94.7, 94.2)
- moved Q1 146.2 mm to (100.4, 90.4)
- moved R1 146.2 mm to (87.2, 111.5)
- moved R2 146.2 mm to (95.4, 89.8)
- moved R3 146.2 mm to (89.8, 89.8)
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Connections:
- C1 pad 2: /HX711/VCC -> +3V3
- J2 pad 1: /HX711/VCC -> Net-(J2-Pad1)
- Q1 pad 2: /HX711/VCC -> +3V3
- R6 pad 1: Net-(JP2-Pad2) -> Net-(JP4-Pad1)
- U2 pad 15: Net-(U2-Pad15) -> GND
- U2 pad 3: Net-(U2-Pad3) -> Net-(R6-Pad2)
- U2 pad 8: Net-(U2-Pad8) -> Net-(JP4-Pad1)
- U3 pad 1: /HX711/VCC -> +3V3
- U3 pad 16: /HX711/VCC -> +3V3
- U_DEMUX1 pad 9: Net-(R6-Pad2) -> Net-(U_DEMUX1-Pad9)
- XA1 pad 41: +3V3 -> +5V
- XA1 pad 42: +5V -> +3V3
Other:
- board outline removed

Commit message: update files
Parts:
- removed the MP? at (133.9, 97.3)
- added C4: 100nF, Capacitor_SMD:C_1206_3216Metric_Pad1.33x1.80mm_HandSolder, F.Cu at (112.1, 58.5)
- added J1: Conn_01x16_Female, Connector_PinHeader_2.54mm:PinHeader_1x16_P2.54mm_Vertical, F.Cu at (72.4, 136.1)
- added J3: Conn_01x16_Female, Connector_PinHeader_2.54mm:PinHeader_1x16_P2.54mm_Vertical, F.Cu at (126.4, 97.4)
- added J4: Conn_01x01_Male, Connector_PinHeader_2.54mm:PinHeader_1x01_P2.54mm_Vertical, F.Cu at (121.5, 57.9)
- added J5: Conn_01x01_Male, Connector_PinHeader_2.54mm:PinHeader_1x01_P2.54mm_Vertical, F.Cu at (96.8, 93.2)
- added J6: Conn_01x01_Male, Connector_PinHeader_2.54mm:PinHeader_1x01_P2.54mm_Vertical, F.Cu at (69.7, 56.6)
- added MP?: Plantilla_EDU-CIAA, celda:Plantilla_EDU-CIAA, F.Cu at (133.9, 97.3)
- C1, C2, C3: footprint Capacitor_THT:CP_Radial_D4.0mm_P1.50mm -> Capacitor_SMD:C_1206_3216Metric_Pad1.33x1.80mm_HandSolder
- Q1: footprint Package_TO_SOT_SMD:SOT-23 -> Connector_PinHeader_2.54mm:PinHeader_1x02_P2.54mm_Vertical
- SW1, SW2: value SW_MEC_5G -> SW_MEC_5E
- U_DEMUX1, U_MUX1: value CD74HC4067M -> CD74HC4067SM; footprint Package_SO:SOIC-24W_7.5x15.4mm_P1.27mm -> Package_SO:SSOP-24_5.3x8.2mm_P0.65mm
- moved U3 47.6 mm to (84.8, 73.7)
- moved R4 41.4 mm to (86.7, 106.6), turned to 90 degrees
- moved U_MUX1 37.5 mm to (112.3, 117.6), turned to 270 degrees
- moved JP6 36.4 mm to (122.7, 87.8), turned to 180 degrees
- moved C3 35.6 mm to (69.7, 68.8), turned to 90 degrees
- moved C1 35.4 mm to (74.8, 61.8)
- moved R5 34.8 mm to (102.9, 124.5), turned to 180 degrees
- moved SW2 33.9 mm to (102.7, 91.7)
- moved J2 33.8 mm to (63.5, 59.4)
- moved Q1 33.3 mm to (76.7, 67.1), turned to 180 degrees
- moved JP7 33.0 mm to (116.7, 89.3), turned to 180 degrees
- moved JP8 32.4 mm to (84.2, 93.6), turned to 270 degrees
- moved R1 30.6 mm to (72.1, 84.9), turned to 90 degrees
- moved R6 27.2 mm to (104.8, 59.1)
- moved R2 26.5 mm to (75.7, 72.1)
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Connections:
- net Net-(XA1-Pad27) renamed /Conector-EDU_CIAA/CAN_RD-GPIO33
- net Net-(XA1-Pad29) renamed /Conector-EDU_CIAA/CAN_TD-GPIO32
- net Net-(XA1-Pad31) renamed /Conector-EDU_CIAA/T_COL1-GPIO30
- C1 pad 2: +3V3 -> /HX711/VCC
- JP1 pad 2: Net-(JP1-Pad2) -> +5V
- JP2 pad 2: Net-(JP2-Pad2) -> +5V
- JP3 pad 1: Net-(C4-Pad1) -> /HX711/VCC
- JP3 pad 2: /NodeMCU/RST -> +5V
- JP4 pad 1: Net-(JP4-Pad1) -> +3V3
- JP4 pad 2: +3V3 -> /NodeMCU/+3V3
- JP5 pad 1: Net-(JP5-Pad1) -> /HX711/SCK
- JP5 pad 2: /NodeMCU/GPIO0 -> /Conector-EDU_CIAA/RXD1-GPIO21
- JP6 pad 1: Net-(JP6-Pad1) -> /Conector-EDU_CIAA/232_RX
- JP6 pad 2: /Conector-EDU_CIAA/232_RX -> /NodeMCU/TX
- JP7 pad 1: Net-(JP7-Pad1) -> /Conector-EDU_CIAA/232_TX
- JP7 pad 2: /Conector-EDU_CIAA/232_TX -> /NodeMCU/RX
- JP8 pad 1: GND -> /HX711/DT
- JP8 pad 2: GND -> /Conector-EDU_CIAA/TX_EN-GPIO19
- Q1 pad 2: +3V3 -> /HX711/VCC
- R10 pad 1: Net-(JP4-Pad1) -> /NodeMCU/+3V3
- R6 pad 1: Net-(JP4-Pad1) -> /NodeMCU/+3V3
- R7 pad 1: Net-(JP4-Pad1) -> /NodeMCU/+3V3
- R7 pad 2: Net-(C4-Pad1) -> /NodeMCU/RST
- R8 pad 1: Net-(JP4-Pad1) -> /NodeMCU/+3V3
- R8 pad 2: Net-(JP5-Pad1) -> /NodeMCU/GPIO0-D3
- SW1 pad 1: GND -> /NodeMCU/RST
- SW1 pad 2: GND -> /NodeMCU/RST
- SW2 pad 1: Net-(JP5-Pad1) -> /NodeMCU/GPIO0-D3
- SW2 pad 2: Net-(JP5-Pad1) -> /NodeMCU/GPIO0-D3
- U2 pad 1: Net-(C4-Pad1) -> /NodeMCU/RST
- U2 pad 18: Net-(JP5-Pad1) -> /NodeMCU/GPIO0-D3
- U2 pad 21: Net-(JP7-Pad1) -> /NodeMCU/RX
- U2 pad 22: Net-(JP6-Pad1) -> /NodeMCU/TX
- U2 pad 8: Net-(JP4-Pad1) -> /NodeMCU/+3V3
- U3 pad 1: +3V3 -> /HX711/VCC
- U3 pad 16: +3V3 -> /HX711/VCC
- U_DEMUX1 pad 1: Net-(U_DEMUX1-Pad1) -> /Conector-EDU_CIAA/GPIO8
- U_DEMUX1 pad 10: Net-(U_DEMUX1-Pad10) -> /Conector-EDU_CIAA/GPIO1
- U_DEMUX1 pad 11: Net-(U_DEMUX1-Pad11) -> /Conector-EDU_CIAA/GPIO3
- U_DEMUX1 pad 13: Net-(U_DEMUX1-Pad13) -> /Conector-EDU_CIAA/GPIO7
- U_DEMUX1 pad 14: Net-(U_DEMUX1-Pad14) -> /Conector-EDU_CIAA/GPIO5
- U_DEMUX1 pad 15: Net-(R5-Pad1) -> Net-(R4-Pad1)
- U_DEMUX1 pad 16: Net-(U_DEMUX1-Pad16) -> GND
- U_DEMUX1 pad 17: Net-(U_DEMUX1-Pad17) -> GND
- U_DEMUX1 pad 24: Net-(JP2-Pad1) -> Net-(JP1-Pad1)
- U_MUX1 pad 1: Net-(U_MUX1-Pad1) -> /Conector-EDU_CIAA/CH3
- U_MUX1 pad 10: Net-(U_MUX1-Pad10) -> /Conector-EDU_CIAA/T_FIL0-GPIO25
- U_MUX1 pad 11: Net-(U_MUX1-Pad11) -> /Conector-EDU_CIAA/T_FIL3-GPIO28
- U_MUX1 pad 13: Net-(U_MUX1-Pad13) -> /Conector-EDU_CIAA/T_COL0-GPIO29
- U_MUX1 pad 14: Net-(U_MUX1-Pad14) -> /Conector-EDU_CIAA/T_FIL2-GPIO27
- U_MUX1 pad 15: Net-(R4-Pad1) -> Net-(R5-Pad1)
- U_MUX1 pad 16: Net-(U_MUX1-Pad16) -> GND
- U_MUX1 pad 17: Net-(U_MUX1-Pad17) -> GND
- U_MUX1 pad 18: Net-(U_MUX1-Pad18) -> GND
- U_MUX1 pad 19: Net-(U_MUX1-Pad19) -> GND
- U_MUX1 pad 24: Net-(JP1-Pad1) -> Net-(JP2-Pad1)
- XA1 pad 2: +5V -> /Conector-EDU_CIAA/+5V_P1
- XA1 pad 33: Net-(XA1-Pad33) -> /Conector-EDU_CIAA/T_FIL0-GPIO25
- XA1 pad 35: Net-(XA1-Pad35) -> /Conector-EDU_CIAA/T_FIL3-GPIO28
- XA1 pad 37: Net-(XA1-Pad37) -> /Conector-EDU_CIAA/T_FIL2-GPIO27
- XA1 pad 39: Net-(XA1-Pad39) -> /Conector-EDU_CIAA/T_COL0-GPIO29
- XA1 pad 41: +5V -> /Conector-EDU_CIAA/+3.3V_P2
- XA1 pad 42: +3V3 -> +5V
- XA1 pad 44: Net-(XA1-Pad44) -> /Conector-EDU_CIAA/RXD1-GPIO21
- XA1 pad 46: Net-(XA1-Pad46) -> /Conector-EDU_CIAA/TX_EN-GPIO19
Routing:
- net GND: track 0.00 -> 154.9 mm, vias 0 -> 10
- net +5V: track 0.00 -> 93.0 mm, vias 0 -> 1
- net +3V3: track 0.00 -> 65.6 mm, vias 0 -> 1
- net /NodeMCU/+3V3: track 0.00 -> 58.3 mm, vias 0 -> 1
- net /Conector-EDU_CIAA/T_FIL3-GPIO28: track 0.00 -> 55.0 mm, vias 0 -> 2
- net /Conector-EDU_CIAA/CH3: track 0.00 -> 53.4 mm, vias 0 -> 2
- net /Conector-EDU_CIAA/232_TX: track 0.00 -> 51.0 mm, vias 0 -> 1
- net /Conector-EDU_CIAA/GPIO8: track 0.00 -> 49.8 mm
- net /Conector-EDU_CIAA/T_FIL0-GPIO25: track 0.00 -> 49.7 mm, vias 0 -> 2
- net /NodeMCU/RST: track 0.00 -> 46.7 mm, vias 0 -> 2
- net /Conector-EDU_CIAA/232_RX: track 0.00 -> 45.7 mm, vias 0 -> 1
- net /Conector-EDU_CIAA/GPIO5: track 0.00 -> 45.4 mm, vias 0 -> 2
- net /Conector-EDU_CIAA/GPIO7: track 0.00 -> 43.4 mm, vias 0 -> 2
- net /HX711/E+: track 0.00 -> 43.2 mm, vias 0 -> 1
- net /Conector-EDU_CIAA/T_COL0-GPIO29: track 0.00 -> 39.1 mm
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- added copper zone on F.Cu, net GND

Commit message: Update files
Parts:
- SW1, SW2: value SW_MEC_5E -> SW_Push
- moved SW1 8.03 mm to (90.3, 61.9), turned to 180 degrees
- moved SW2 1.67 mm to (101.1, 91.9)
- moved C1 1.45 mm to (75.1, 60.5)
Connections:
- SW1 pad 1: /NodeMCU/RST -> GND
- SW2 pad 2: /NodeMCU/GPIO0-D3 -> GND
Routing:
- net GND: track 154.9 -> 184.4 mm, vias 10 -> 15
- net /Conector-EDU_CIAA/GPIO5: track 45.4 -> 51.5 mm
- net /Conector-EDU_CIAA/GPIO7: track 43.4 -> 49.2 mm
- net /HX711/VCC: track 29.7 -> 33.7 mm
- net /HX711/E+: track 43.2 -> 40.8 mm
- net /NodeMCU/GPIO0-D3: track 25.4 -> 27.2 mm
- net /Conector-EDU_CIAA/GPIO1: track 32.3 -> 34.0 mm
- net Net-(Q1-Pad1): track 5.65 -> 7.35 mm, vias 0 -> 1
- net /Conector-EDU_CIAA/GPIO3: track 32.7 -> 34.4 mm
- net Net-(J1-Pad1): track 20.7 -> 22.2 mm, vias 0 -> 1
- net /Conector-EDU_CIAA/GPIO8: track 49.8 -> 50.9 mm
- net Net-(J1-Pad2): track 18.7 -> 19.7 mm, vias 0 -> 1
- net Net-(J1-Pad7): track 12.8 -> 11.9 mm, vias 0 -> 1
- net Net-(J1-Pad8): track 13.4 -> 12.6 mm, vias 0 -> 1
- net Net-(J1-Pad3): track 16.7 -> 17.5 mm, vias 0 -> 1
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
Commit message: Update files
Parts:
- added C5: 10uF, Capacitor_SMD:C_1206_3216Metric_Pad1.33x1.80mm_HandSolder, F.Cu at (69.8, 62.5)
- added C6: 100nF, Capacitor_SMD:C_1206_3216Metric_Pad1.33x1.80mm_HandSolder, F.Cu at (88.6, 82.6)
- added R11: 1.2k, Resistor_SMD:R_1206_3216Metric, F.Cu at (92.2, 82.5)
- Q1: footprint Connector_PinHeader_2.54mm:PinHeader_1x02_P2.54mm_Vertical -> Package_TO_SOT_SMD:SOT-23
- moved C1 2.08 mm to (77.1, 61.1)
- moved Q1 0.43 mm to (76.9, 66.7)
Connections:
- U3 pad 10: GND -> Net-(C6-Pad1)
- U3 pad 9: GND -> /HX711/B-
Routing:
- net GND: track 184.4 -> 206.4 mm, vias 15 -> 17
- net Net-(C6-Pad1): track 0.00 -> 11.2 mm
- net /HX711/B-: track 0.00 -> 8.57 mm
- net /HX711/E+: track 40.8 -> 49.2 mm
- net /Conector-EDU_CIAA/GPIO8: track 50.9 -> 57.7 mm
- net /NodeMCU/GPIO0-D3: track 27.2 -> 32.0 mm
- net /HX711/VCC: track 33.7 -> 30.5 mm
- net Net-(Q1-Pad1): track 7.35 -> 5.66 mm, vias 1 -> 0
- net /HX711/E-: track 31.3 -> 33.0 mm

Commit message: Update files + gerbers
Parts:
- added C7: C, Capacitor_SMD:C_1206_3216Metric_Pad1.33x1.80mm_HandSolder, F.Cu at (90.2, 106.7)
- added C8: C, Capacitor_SMD:C_1206_3216Metric_Pad1.33x1.80mm_HandSolder, F.Cu at (96.0, 125.7)
- added R12: 1k, Resistor_SMD:R_1206_3216Metric, F.Cu at (125.3, 135.9)
- added R13: 1k, Resistor_SMD:R_1206_3216Metric, F.Cu at (125.3, 133.3)
- added R14: 1k, Resistor_SMD:R_1206_3216Metric, F.Cu at (125.2, 130.8)
- added R15: 1k, Resistor_SMD:R_1206_3216Metric, F.Cu at (125.3, 128.2)
- added R16: 1k, Resistor_SMD:R_1206_3216Metric, F.Cu at (125.3, 125.6)
- added R17: 1k, Resistor_SMD:R_1206_3216Metric, F.Cu at (125.3, 122.9)
- added R18: 1k, Resistor_SMD:R_1206_3216Metric, F.Cu at (125.3, 120.4)
- added R19: 1k, Resistor_SMD:R_1206_3216Metric, F.Cu at (125.4, 117.8)
- added R20: 1k, Resistor_SMD:R_1206_3216Metric, F.Cu at (125.3, 115.2)
- added R21: 1k, Resistor_SMD:R_1206_3216Metric, F.Cu at (125.3, 112.7)
- added R22: 1k, Resistor_SMD:R_1206_3216Metric, F.Cu at (125.2, 110.2)
- added R23: 1k, Resistor_SMD:R_1206_3216Metric, F.Cu at (125.2, 107.5)
- added R24: 1k, Resistor_SMD:R_1206_3216Metric, F.Cu at (125.2, 105.0)
- added R25: 1k, Resistor_SMD:R_1206_3216Metric, F.Cu at (125.2, 102.5)
- added R26: 1k, Resistor_SMD:R_1206_3216Metric, F.Cu at (125.1, 99.8)
- added R27: 1k, Resistor_SMD:R_1206_3216Metric, F.Cu at (125.1, 97.1)
- moved JP1 16.3 mm to (96.3, 102.4), turned to 270 degrees
- moved J3 9.02 mm to (117.3, 97.5)
- moved JP2 8.19 mm to (94.5, 114.6)
- moved R5 8.18 mm to (96.1, 129.0)
- moved U_MUX1 7.37 mm to (104.9, 117.9)
Connections:
- J3 pad 13: GND -> Net-(J3-Pad13)
- J3 pad 14: GND -> Net-(J3-Pad14)
- J3 pad 15: GND -> Net-(J3-Pad15)
- J3 pad 16: GND -> Net-(J3-Pad16)
- R5 pad 2: GND -> GNDA
- U_MUX1 pad 12: GND -> GNDA
- U_MUX1 pad 16: GND -> Net-(J3-Pad16)
- U_MUX1 pad 17: GND -> Net-(J3-Pad15)
- U_MUX1 pad 18: GND -> Net-(J3-Pad14)
- U_MUX1 pad 19: GND -> Net-(J3-Pad13)
- XA1 pad 18: Net-(XA1-Pad18) -> GNDA
Routing:
- net GNDA: track 0.00 -> 156.4 mm, vias 0 -> 3
- net GND: track 206.4 -> 102.8 mm, vias 17 -> 9
- net Net-(J3-Pad16): track 0.00 -> 34.8 mm, vias 0 -> 2
- net Net-(J3-Pad15): track 0.00 -> 31.1 mm, vias 0 -> 2
- net Net-(J3-Pad14): track 0.00 -> 27.6 mm, vias 0 -> 2
- net Net-(J3-Pad13): track 0.00 -> 24.8 mm, vias 0 -> 2
- net /Conector-EDU_CIAA/T_COL0-GPIO29: track 39.1 -> 55.4 mm
- net /Conector-EDU_CIAA/T_FIL2-GPIO27: track 36.3 -> 50.7 mm
- net Net-(C7-Pad1): track 19.2 -> 32.9 mm
- net Net-(C8-Pad2): track 16.5 -> 30.0 mm
- net /Conector-EDU_CIAA/T_FIL0-GPIO25: track 49.7 -> 62.0 mm
- net /Conector-EDU_CIAA/T_FIL3-GPIO28: track 55.0 -> 65.8 mm
- net Net-(J3-Pad1): track 25.5 -> 33.5 mm, vias 1 -> 2
- net +5V: track 93.0 -> 85.3 mm
- net Net-(J3-Pad2): track 23.2 -> 29.8 mm, vias 1 -> 2
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Other:
- board outline added: 85.9 x 97.3 mm

Commit message: Update files final
Parts:
- moved R9 1.87 mm to (102.6, 84.8), turned to 270 degrees
- moved R7 0.83 mm to (98.6, 58.5), turned to 180 degrees
- moved R6 0.66 mm to (104.9, 58.5)
- moved R10 0.30 mm to (106.1, 84.8)
Routing:
- net GND: track 102.8 -> 108.1 mm
- net /NodeMCU/RST: track 46.7 -> 47.8 mm
- net Net-(J1-Pad13): track 15.9 -> 14.9 mm
- net Net-(J3-Pad15): track 31.1 -> 30.1 mm
- net Net-(J3-Pad14): track 27.6 -> 26.7 mm
- net Net-(J1-Pad14): track 18.2 -> 18.8 mm
- net Net-(J1-Pad7): track 11.9 -> 12.5 mm

Commit message: Ultimos detalles
Parts:
- moved R7 2.99 mm to (101.6, 58.2), turned to 90 degrees
- moved R6 1.08 mm to (105.9, 58.2), turned to 90 degrees
- moved C4 0.63 mm to (112.6, 58.1), turned to 90 degrees
Routing:
- net Net-(R6-Pad2): track 8.91 -> 10.8 mm
